File: atsaml10-breakout.kicad_pcb (KiCad board)
At the start: 2 copper layers, 25.4 x 50.8 mm, 40 parts, among them J1 Conn_01x16, J2 Conn_01x16, J3 SWD, Q1 BC847, Q2 BC847, SW1 Reset, U1 ATSAML10E16A-A, Y1 32.768kHz, Y2 8MHz

Commit message: Replaced L1's footprint with Coilcraft LPS3015
Parts:
- L1: footprint Inductor_SMD:L_0603_1608Metric -> Elevendroids_Inductor_SMD:L_Coilcraft_LPS3015
- moved C7 0.76 mm to (124.2, 68.1)
- moved R7 0.76 mm to (122.7, 68.1)
- moved R8 0.76 mm to (125.7, 68.1)
- moved L1 0.46 mm to (121.2, 82.7), turned to 180 degrees
Routing:
- net /~RESET: track 44.4 -> 43.0 mm
- net Net-(L1-Pad2): track 8.36 -> 7.10 mm
- net VDD: track 105.8 -> 104.6 mm
- net Net-(C8-Pad1): track 7.64 -> 8.81 mm

Commit message: More layout tweaks
Parts:
- moved R2 38.2 mm to (147.1, 95.5)
- moved R4 38.2 mm to (148.6, 95.5)
- moved J2 38.0 mm to (162.8, 123.2)
- moved Y1 37.8 mm to (149.4, 92.7)
- moved C11 37.8 mm to (152.3, 98.9)
- moved C10 37.8 mm to (150.6, 113.0)
- moved C3 37.8 mm to (153.2, 116.8)
- moved D2 37.8 mm to (147.1, 123.4)
- moved FB1 37.8 mm to (147.1, 113.0)
- moved J1 37.8 mm to (142.2, 85.1)
- moved J3 37.8 mm to (152.4, 86.4)
- moved Q2 37.8 mm to (146.3, 123.4)
- moved R13 37.8 mm to (145.5, 120.1)
- moved R14 37.8 mm to (151.1, 120.1)
- moved R15 37.8 mm to (147.1, 120.1)
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Routing:
- net /PA30_SWCLK: track 26.9 -> 28.8 mm
- net GND: track 1.67 -> 0.00 mm, vias 18 -> 29
- net /~RESET: track 43.0 -> 44.5 mm
- net /PA00: track 16.2 -> 17.6 mm
- net /PA00_XIN32: track 9.67 -> 11.1 mm
- net /PA01_XOUT32: track 10.0 -> 11.2 mm
- net Net-(C8-Pad1): track 8.81 -> 8.27 mm
- net /PA01: track 7.99 -> 8.49 mm
Other:
- board size 25.4 x 50.8 mm -> 24.4 x 50.8 mm
- net class Power added: clearance 0.2, trace_width 0.5, via_dia 0.8, via_drill 0.4
- net class VDD removed
